File: MotorCAN/MotorCAN.kicad_sch (KiCad schematic)
At the start: 48 parts, among them CN1 ZX-SH1.0-3PWT, CN2 HCZZ0021-4, CN3 HCZZ0021-4, J1 MTR, U1 STM32G431CBT6, U2 DRV8316CRRGFR, U3 TCAN330GDCNR, U4 MT6816CT-AKD-R, X1 XL7EL89CKI-111YLC-24M

Commit message: Added finalized design, with some issues fixed
Parts:
- removed CN2, CN3: HCZZ0021-4, easyeda2kicad:CONN-SMD_HCZZ0021-4, symbol easyeda2kicad:HCZZ0021-4
- removed J1: MTR, Connector_PinHeader_2.54mm:PinHeader_1x03_P2.54mm_Vertical, symbol Connector:Conn_01x03_Pin
- removed TP2: 3V3, TestPoint:TestPoint_Pad_D1.0mm, symbol Connector:TestPoint_Probe
- removed TP3: VIN, TestPoint:TestPoint_Pad_D1.0mm, symbol Connector:TestPoint_Probe
- removed U3: TCAN330GDCNR, easyeda2kicad:SOT-23-8_L2.9-W1.6-P0.65-LS2.8-BL, symbol easyeda2kicad:TCAN330GDCNR
- added C27, C28: 100nF, Capacitor_SMD:C_0402_1005Metric, symbol Device:C_Small
- added C29: 100uF, Capacitor_SMD:CP_Elec_6.3x7.7, symbol Device:C_Small
- added CN2, CN3: WAFER-GH1.25-4PWB, easyeda2kicad:CONN-SMD_4P-P1.25_XUNPU_WAFER-GH1.25-4PWB, symbol easyeda2kicad:WAFER-GH1.25-4PWB
- added CN4, CN5, CN6: ZX-SH1.0-3PWT, easyeda2kicad:CONN-SMD_3P-P1.00_MEGASTAR_ZX-SH1.0-3PWT, symbol easyeda2kicad:ZX-SH1.0-3PWT
- added H1, H3, H4: MountingHole_Pad, MountingHole:MountingHole_2.2mm_M2_ISO14580_Pad_TopBottom, symbol Mechanical:MountingHole_Pad
- added J2: PWR IN, Connector_AMASS:AMASS_XT30PW-M_1x02_P2.50mm_Horizontal, symbol Connector:Conn_01x02_Pin
- added J3: PWR OUT, Connector_AMASS:AMASS_XT30PW-F_1x02_P2.50mm_Horizontal, symbol Connector:Conn_01x02_Socket
- added M1: A, Connector_Wire:SolderWirePad_1x01_SMD_2x4mm, symbol Connector:Conn_01x01_Pin
- added M2: B, Connector_Wire:SolderWirePad_1x01_SMD_2x4mm, symbol Connector:Conn_01x01_Pin
- added M3: C, Connector_Wire:SolderWirePad_1x01_SMD_2x4mm, symbol Connector:Conn_01x01_Pin
- added Q1: 2N7002, Package_TO_SOT_SMD:SOT-23, symbol Transistor_FET:2N7002
- added R10, R11, R13, R14, R9: 10k, Resistor_SMD:R_0603_1608Metric, symbol Device:R_Small_US
- added R12, R7: 100k, Resistor_SMD:R_0603_1608Metric, symbol Device:R_Small_US
- added R8: 100, Resistor_SMD:R_0603_1608Metric, symbol Device:R_Small_US
- added U3: SN65HVD230DR, easyeda2kicad:SOIC-8_L4.9-W3.9-P1.27-LS6.0-BL, symbol easyeda2kicad:SN65HVD230DR
- C10, C11, C12, C3, C4, C5, C6, C7, C8, C9: footprint Capacitor_SMD:C_0805_2012Metric -> Capacitor_SMD:C_1206_3216Metric
- D3: value 18V -> 26V; footprint Diode_SMD:D_SMA -> Diode_SMD:D_SMB
- R1: now fitted
Connections:
- net 3V3 is gone; now on net +3V3: C16.1, U4.2 (HVPP), U4.4 (VDD)
- net +3V3: now also U2.28 (INLA), U2.30 (INLB), U2.32 (INLC), U2.37 (VREF/ILIM), CN4.1, R10.1, R11.1, R14.2, U3.3 (VCC)
- net CSENC: now also U1.22 (PB10), R11.2; no longer U1.43 (PB6)
- net DRVOFF: now also R14.1
- net GND: now also U2.12 (PGND), U2.15 (PGND), U2.18 (PGND), C27.1, C28.2, C29.2, CN2.4, CN3.4, CN4.3, CN5.2, CN6.2, H1.1, H3.1, H4.1, J2.1 (Pin_1), J3.1 (Pin_1), Q1.2 (S), R13.2, R7.2, R9.2, U3.2 (GND), U3.8 (RS)
- net MISO2: now also U1.28 (PB14); no longer U1.41 (PB4)
- net MOSI2: now also U1.29 (PB15); no longer U1.42 (PB5)
- net OUTA: now also M1.1 (Pin_1)
- net OUTB: now also M2.1 (Pin_1)
- net OUTC: now also M3.1 (Pin_1)
- net RXD: now also U3.4 (R)
- net SPICLK2: now also U1.27 (PB13); no longer U1.40 (PB3)
- net SWCLK: now also CN6.1
- net SWDIO: now also CN6.3; no longer CN1.1
- net TXD: now also U3.1 (D)
- net VIN: now also C29.1, J2.2 (Pin_2), J3.2 (Pin_2), R12.1
- net nSCS: now also U1.25 (PB11), R10.2; no longer U1.11 (PA3)
- net at D1.1 (K), R2.2, R3.1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: now also Q1.3 (D)
- net DEBUG: now reaches U1.12 (PA4)
- net HALL: now reaches U1.16 (PB0)
- net HALL: now also CN4.2
- net at U1.2 (PC13): now also R8.2
- net UART1RX: now reaches U1.44 (PB7)
- net UART1RX: now also CN1.1
- net at U1.45 (PB8-BOOT0): now also R9.1
- net NRST: now reaches U1.7 (PG10-NRST)
- net NRST: now also C27.2, CN5.1
- net CANH renamed CAN+
- net CAN+: now also CN2.2, CN3.2, U3.7 (CANH)
- net CANL renamed CAN-
- net CAN-: now also CN2.3, CN3.3, U3.6 (CANL)
- removed net INAL: U1.27 (PB13), U2.28 (INLA)
- removed net INBL: U1.28 (PB14), U2.30 (INLB)
- removed net INCL: U1.29 (PB15), U2.32 (INLC)
- net SWDCLK renamed UART1TX
- net UART1TX: now also U1.43 (PB6)
- new net RST: Q1.1 (G), R7.1, R8.1
- new net SWO: CN5.3, U1.40 (PB3)
- new net VREAD: C28.1, R12.2, R13.1, U1.11 (PA3)
- no-connect marks 0 -> 27
Other:
- moved on the sheet: C14
